File: unisplit_orthosteno.kicad_sch (KiCad schematic)
At the start: 58 parts, among them SW1 SW_SPST, U1 ProMicro

Commit message: feat(mcu): swap Pro Micro for KB2040 in the schematic
Repoints U1 at uni-symbols:KB2040 and renames pins to their RP2040
functions. Pin numbers and pin coordinates are unchanged, so every wire,
junction and global label stays attached; the matrix netlist is
untouched.

Renames the +5V rail to +3V3. KB2040 pad 21 is a 3.3 V regulator output,
not a 5 V rail, and is now typed power_out accordingly. The rail drives
nothing but the passive diode matrix, so this is an accurate relabelling
rather than a circuit change.

Pad 24 (RAW) is now typed power_in instead of input. It remains
unconnected, as on the Pro Micro; per Adafruit's schematic the module
self-powers from USB through D1 into regulator U2.

Verified against a netlist export before and after: 50 nets and 138
nodes in both, no net changed membership, and the connectivity graph is
identical. ERC 133 -> 70.
Parts:
- U1: value ProMicro -> KB2040; footprint Keebio-Parts:ArduinoProMicro -> uni-footprints:Adafruit_KB2040; symbol keebio:ProMicro -> uni-symbols:KB2040
Connections:
- net +5V renamed +3V3
Changed lines of the file:
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@@
     (pin "2")
   )
-  (symbol (lib_id "keebio:ProMicro") (at 139.7 121.92 0) (mirror y) (unit 1)
+  (symbol (lib_id "uni-symbols:KB2040") (at 139.7 121.92 0) (mirror y) (unit 1)
     (in_bom yes) (on_board yes)
     (property "Reference" "U1" (id 0) (at 139.7 100.6602 0)
       (effects (font (size 1.524 1.524)))
     )
-    (property "Value" "ProMicro" (id 1) (at 139.7 103.3526 0)
-      (effects (font (size 1.524 1.524)))
-    )
-    (property "Footprint" "Keebio-Parts:ArduinoProMicro" (id 2) (at 113.03 185.42 90)
+    (property "Value" "KB2040" (id 1) (at 139.7 103.3526 0)
+      (effects (font (size 1.524 1.524)))
+    )
+    (property "Footprint" "uni-footprints:Adafruit_KB2040" (id 2) (at 113.03 185.42 90)
       (effects (font (size 1.524 1.524)) hide)
     )
@@
     (pin "1")
   )
-  (symbol (lib_id "unisplit_orthosteno-rescue:+5V-power") (at 100.33 115.57 0) (unit 1)
+  (symbol (lib_id "unisplit_orthosteno-rescue:+3V3-power") (at 100.33 115.57 0) (unit 1)
     (in_bom yes) (on_board yes)
     (property "Reference" "#PWR0104" (id 0) (at 100.33 119.38 0)
       (effects (font (size 1.27 1.27)) hide)
     )
-    (property "Value" "+5V" (id 1) (at 100.711 111.1758 0))
+    (property "Value" "+3V3" (id 1) (at 100.711 111.1758 0))
     (property "Footprint" "" (id 2) (at 100.33 115.57 0)
       (effects (font (size 1.27 1.27)) hide)
@@
     )
     (path "/00000000-0000-0000-0000-00006010d314"
-      (reference "#PWR0104") (unit 1) (value "+5V") (footprint "")
+      (reference "#PWR0104") (unit 1) (value "+3V3") (footprint "")
     )
     (path "/981ca761-e4a5-456a-aa1e-bf708f8eb19e"
@@
     )
     (path "/00000000-0000-0000-0000-000060091c15"
-      (reference "U1") (unit 1) (value "ProMicro") (footprint "Keebio-Parts:ArduinoProMicro")
-    )
-  )
+      (reference "U1") (unit 1) (value "KB2040") (footprint "uni-footprints:Adafruit_KB2040")
+    )
+  )
