File: unisplit_orthosteno.kicad_pcb (KiCad board)
At the start: 2 copper layers, 247.6 x 76.2 mm, 65 parts, among them SW1 SW_SPST, U1 ProMicro

Commit message: feat(mcu): swap Pro Micro footprint for KB2040 on the PCB
Replaces the Keebio-Parts:ArduinoProMicro footprint at U1 with
uni-footprints:Adafruit_KB2040. All 24 pads keep their exact
coordinates, sizes, drills, nets and tstamps, so no track moved.
Silkscreen labels become RP2040 GPIO numbers; they are bare numerals
because board setup enforces a 0.8 mm minimum text height, at which
four characters do not fit on the 2.54 mm pad pitch.

Adds an F/B courtyard, which the Pro Micro footprint lacked, and
replaces the micro-USB outline on Dwgs.User with the USB-C mechanical
envelope measured from Adafruit's board file. The connector is 1.570 mm
wider and sits 0.317 mm further inside the board edge, so the case
opening needs widening.

Updates the assembly silkscreen from "pro micro on this side" to
"kb2040 on this side".

DRC 239 -> 181: zero new violations, 58 resolved. Every remaining
violation attributes to a pre-existing footprint and none to U1. Bytes
before and after the footprint block are unchanged, and track, via,
zone, net and Edge.Cuts counts all match.
Parts:
- U1: value ProMicro -> KB2040; footprint Keebio-Parts:ArduinoProMicro -> uni-footprints:Adafruit_KB2040
Other:
- board text added: "kb2040 on this side smooth side up"
- board text removed: "pro micro on this side smooth side up"

Commit message: fix(pcb): name the KB2040 logic rail +3V3 to match the schematic
The schematic drives U1 pad 21 from a +3V3 power symbol, and the pad already
carries pinfunction "3V3" / pintype "power_out", but the board file still
declared and referenced net 45 as "+5V" - the Pro Micro name it inherited. The
generated gerbers inherited it too, emitting %TO.N,+5V*% for that pad.

Net 45 has a single node (U1 pad 21) and no tracks, so this is a rename with no
connectivity change. Verified against a netlist export of the schematic: the
only PCB/schematic net-name mismatch on a PR-touched node was this one, and DRC
is unchanged at 230 violations with 0 unconnected items before and after.

Gerbers and drill files regenerated with the same KiCad 10.0.5 settings as the
previous export (X2, 4.6 mm, protel extensions, soldermask subtracted from
silkscreen; excellon inch/decimal/absolute, separate PTH and NPTH). Diffed
against the committed set ignoring timestamps, the only substantive change is
%TO.N,+5V*% -> %TO.N,+3V3*% in F_Cu.gtl and B_Cu.gbl; every other layer and
both drill files are byte-identical.
Connections:
- net +5V renamed +3V3
Changed lines of the file:
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@@
   (net 43 "unconnected-(U1-Pad5)")
   (net 44 "unconnected-(U1-Pad6)")
-  (net 45 "+5V")
+  (net 45 "+3V3")
   (net 46 "reset")
   (net 47 "unconnected-(U1-Pad24)")
@@
       (net 1 "row0") (pinfunction "A3/GPIO29") (pintype "bidirectional"))
     (pad "21" thru_hole circle locked (at -6.35 7.62 270) (size 1.7526 1.7526) (drill 1.0922) (layers *.Cu *.SilkS *.Mask)
-      (net 45 "+5V") (pinfunction "3V3") (pintype "power_out"))
+      (net 45 "+3V3") (pinfunction "3V3") (pintype "power_out"))
     (pad "22" thru_hole circle locked (at -8.89 7.62 270) (size 1.7526 1.7526) (drill 1.0922) (layers *.Cu *.SilkS *.Mask)
       (net 46 "reset") (pinfunction "RST") (pintype "input"))
